Commit message: update piper sdk and teleop collect support.

File: third_party/agilex-arm-gravity-compensation/piper_description/urdf/piper_description_with_teach.urdf (robot description, URDF)
Before this commit: robot piper, 10 links, 9 joints
Links:
- link link7: mass 0.02 -> 0.04
- link link8: mass 0.02 -> 0.04
- link teach_base: mass 0.5 -> 0.6
